File: pcb/fpga-dev.kicad_sch (KiCad schematic)
At the start: 1 part, among them U1 XC6SLX9-TQG144

Commit message: Link fpga part
Parts:
- U1: LCSC (none) -> C27408
Changed lines of the file:
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@@
+			)
+		)
+		(property "LCSC" "C27408"
+			(at 68.58 154.94 0)
+			(effects
+				(font
+					(size 1.27 1.27)
+				)
+				(hide yes)
 			)
 		)
@@
 			)
 		)
+		(property "LCSC" "C27408"
+			(at 212.09 156.21 0)
+			(effects
+				(font
+					(size 1.27 1.27)
+				)
+				(hide yes)
+			)
+		)
 		(pin "68"
 		)
@@
 			)
 		)
+		(property "LCSC" "C27408"
+			(at 83.82 68.58 0)
+			(effects
+				(font
+					(size 1.27 1.27)
+				)
+				(hide yes)
+			)
+		)
 		(pin "68"
 		)
@@
 			(at 231.14 67.31 0)
 			(effects
+				(font
+					(size 1.27 1.27)
+				)
+				(hide yes)
+			)
+		)
+		(property "LCSC" "C27408"
+			(at 231.14 67.31 0)
+			(effects
